File: Wireless-Keyboard.sch (KiCad schematic (older format))
At the start: 155 parts, among them SW1 SW_Push, U1 ATmega32U4-AU, U2 MDBT40, U3 PRTR5V0U2X, Y1 16Mhz

Commit message: mdbt40 circuit
Parts:
- added C?: 1uF, Capacitor_SMD:C_0805_2012Metric, symbol Device:C_Small
- U2: symbol RF_Modules:MDBT40 -> Wireless-Keyboard-rescue:MDBT40-RF_Modules
Connections:
- net GND: now also U2.1 (GND), U2.13 (GND), U2.2 (GND), U2.42 (GND), C?.2
- net VCC: now also U2.14 (VDD), U2.3 (AVDD), C?.1
- no-connect marks 8 -> 10
Other:
- moved on the sheet: U2
Changed lines of the file:
@@
 Connection ~ 7700 6100
 $Comp
-L RF_Modules:MDBT40 U2
+L Wireless-Keyboard-rescue:MDBT40-RF_Modules U2
 U 1 1 5FAAA71F
-P 2975 9475
-F 0 "U2" H 2975 10617 40  0000 C CNN
-F 1 "MDBT40" H 2975 10541 40  0000 C CNN
-F 2 "" H 2625 9725 40  0000 C CNN
-F 3 "" H 2725 9825 40  0000 C CNN
-	1    2975 9475
+P 2950 9450
+F 0 "U2" H 2950 10592 40  0000 C CNN
+F 1 "MDBT40" H 2950 10516 40  0000 C CNN
+F 2 "" H 2600 9700 40  0000 C CNN
+F 3 "" H 2700 9800 40  0000 C CNN
+	1    2950 9450
 	1    0    0    -1
 $EndComp
+$Comp
+L power:GND #PWR?
+U 1 1 5FAB9F44
+P 1650 8200
+F 0 "#PWR?" H 1650 7950 50  0001 C CNN
+F 1 "GND" H 1655 8027 50  0000 C CNN
+F 2 "" H 1650 8200 50  0001 C CNN
+F 3 "" H 1650 8200 50  0001 C CNN
+	1    1650 8200
+	1    0    0    -1
+$EndComp
+Wire Wire Line
+	2100 8850 2100 8750
+Wire Wire Line
+	2100 8750 2100 8200
+Wire Wire Line
+	2100 8200 1650 8200
+Connection ~ 2100 8750
+Wire Wire Line
+	3800 8550 3800 8200
+Wire Wire Line
+	3800 8200 2100 8200
+Connection ~ 2100 8200
+NoConn ~ 3800 8650
+$Comp
+L power:GND #PWR?
+U 1 1 5FB23F96
+P 1500 9250
+F 0 "#PWR?" H 1500 9000 50  0001 C CNN
+F 1 "GND" H 1505 9077 50  0000 C CNN
+F 2 "" H 1500 9250 50  0001 C CNN
+F 3 "" H 1500 9250 50  0001 C CNN
+	1    1500 9250
+	1    0    0    -1
+$EndComp
+$Comp
+L Device:C_Small C?
+U 1 1 5FB5B30D
+P 1650 9250
+F 0 "C?" V 1421 9250 50  0000 C CNN
+F 1 "1uF" V 1512 9250 50  0000 C CNN
+F 2 "Capacitor_SMD:C_0805_2012Metric" H 1650 9250 50  0001 C CNN
+F 3 "~" H 1650 9250 50  0001 C CNN
+	1    1650 9250
+	0    1    1    0
+$EndComp
+Wire Wire Line
+	1550 9250 1500 9250
+Wire Wire Line
+	2100 9250 1850 9250
+$Comp
+L power:VCC #PWR?
+U 1 1 5FBC51B0
+P 1850 9250
+F 0 "#PWR?" H 1850 9100 50  0001 C CNN
+F 1 "VCC" H 1865 9423 50  0000 C CNN
+F 2 "" H 1850 9250 50  0001 C CNN
+F 3 "" H 1850 9250 50  0001 C CNN
+	1    1850 9250
+	1    0    0    -1
+$EndComp
+Connection ~ 1850 9250
+Wire Wire Line
+	1850 9250 1750 9250
+Wire Wire Line
+	2450 10550 2450 10750
+$Comp
+L power:VCC #PWR?
+U 1 1 5FBE2351
+P 2450 10750
+F 0 "#PWR?" H 2450 10600 50  0001 C CNN
+F 1 "VCC" V 2465 10878 50  0000 L CNN
+F 2 "" H 2450 10750 50  0001 C CNN
+F 3 "" H 2450 10750 50  0001 C CNN
+	1    2450 10750
+	0    1    1    0
+$EndComp
+NoConn ~ 2550 10550
+Wire Wire Line
+	2350 10550 1950 10550
+$Comp
+L power:GND #PWR?
+U 1 1 5FC3694C
+P 1950 10550
+F 0 "#PWR?" H 1950 10300 50  0001 C CNN
+F 1 "GND" H 1955 10377 50  0000 C CNN
+F 2 "" H 1950 10550 50  0001 C CNN
+F 3 "" H 1950 10550 50  0001 C CNN
+	1    1950 10550
+	1    0    0    -1
+$EndComp

Commit message: mdbt40 config
Parts:
- added C? (x2): 12pF, Capacitor_SMD:C_0805_2012Metric, symbol Device:C_Small
- added Y?: 32.768KHz, symbol Device:Crystal
- Y1: value 16Mhz -> 16MHz
Connections:
- net GND: now also C?.1, C?.1
- net at U2.10 (P0.27): now also C?.2, Y?.1
- net at U2.9 (P0.26): now also C?.2, Y?.2
Changed lines of the file:
@@
 P 2050 2550
 F 0 "Y1" V 2004 2794 50  0000 L CNN
-F 1 "16Mhz" V 2095 2794 50  0000 L CNN
+F 1 "16MHz" V 2095 2794 50  0000 L CNN
 F 2 "Crystal:Crystal_SMD_3225-4Pin_3.2x2.5mm" H 2050 2550 50  0001 C CNN
 F 3 "~" H 2050 2550 50  0001 C CNN
@@
 	1    0    0    -1
 $EndComp
+$Comp
+L Device:Crystal Y?
+U 1 1 5FC56DDD
+P 1550 10150
+F 0 "Y?" H 1550 9882 50  0000 C CNN
+F 1 "32.768KHz" H 1550 9973 50  0000 C CNN
+F 2 "" H 1550 10150 50  0001 C CNN
+F 3 "~" H 1550 10150 50  0001 C CNN
+	1    1550 10150
+	-1   0    0    1
+$EndComp
+Wire Wire Line
+	2100 9950 1700 9950
+Wire Wire Line
+	1700 9950 1700 10150
+Connection ~ 1700 10150
+Wire Wire Line
+	1700 10150 1700 10350
+Wire Wire Line
+	2100 9850 1400 9850
+Wire Wire Line
+	1400 9850 1400 10150
+Connection ~ 1400 10150
+Wire Wire Line
+	1400 10150 1400 10350
+$Comp
+L Device:C_Small C?
+U 1 1 5FD5832F
+P 1400 10450
+F 0 "C?" V 1171 10450 50  0000 C CNN
+F 1 "12pF" V 1262 10450 50  0000 C CNN
+F 2 "Capacitor_SMD:C_0805_2012Metric" H 1400 10450 50  0001 C CNN
+F 3 "~" H 1400 10450 50  0001 C CNN
+	1    1400 10450
+	-1   0    0    1
+$EndComp
+$Comp
+L Device:C_Small C?
+U 1 1 5FD59789
+P 1700 10450
+F 0 "C?" V 1471 10450 50  0000 C CNN
+F 1 "12pF" V 1562 10450 50  0000 C CNN
+F 2 "Capacitor_SMD:C_0805_2012Metric" H 1700 10450 50  0001 C CNN
+F 3 "~" H 1700 10450 50  0001 C CNN
+	1    1700 10450
+	-1   0    0    1
+$EndComp
+$Comp
+L power:GND #PWR?
+U 1 1 5FD5B3A2
+P 1700 10650
+F 0 "#PWR?" H 1700 10400 50  0001 C CNN
+F 1 "GND" H 1705 10477 50  0000 C CNN
+F 2 "" H 1700 10650 50  0001 C CNN
+F 3 "" H 1700 10650 50  0001 C CNN
+	1    1700 10650
+	1    0    0    -1
+$EndComp
+$Comp
+L power:GND #PWR?
+U 1 1 5FD5B713
+P 1400 10650
+F 0 "#PWR?" H 1400 10400 50  0001 C CNN
+F 1 "GND" H 1405 10477 50  0000 C CNN
+F 2 "" H 1400 10650 50  0001 C CNN
+F 3 "" H 1400 10650 50  0001 C CNN
+	1    1400 10650
+	1    0    0    -1
+$EndComp
+Wire Wire Line
+	1700 10550 1700 10650
+Wire Wire Line
+	1400 10550 1400 10650
 $EndSCHEMATC
